File: OpenESC-20x20-QC/20x20-ESC-QC.kicad_pcb (KiCad board)
At the start: 4 copper layers, 100 x 100 mm, 45 parts

Commit message: chore: consolidate fixture design assets and guidance
Routing:
- removed copper zone on F.Cu, net (none)
